File: hardware/pcb/kicad/patternflow.kicad_pcb (KiCad board)
At the start: 2 copper layers, 74 x 132.5 mm, 35 parts, among them J1 Conn_02x08_Odd_Even, J2 Screw_Terminal_01x02, J3 Screw_Terminal_01x02, SW1 RotaryEncoder_Switch, SW2 RotaryEncoder_Switch, SW3 RotaryEncoder_Switch, SW4 RotaryEncoder_Switch, U1 ESP32-S3-DevKit-44pin

Commit message: GPIO0 pullup fix, encoder silkscreen fix
Parts:
- removed C11: 1000uF/16V, Capacitor_THT:CP_Radial_D10.0mm_P5.00mm
- added R13: 10k, Resistor_SMD:R_0805_2012Metric_Pad1.20x1.40mm_HandSolder, F.Cu at (98.5, 130.5)
Connections:
- U1 pad 36: unconnected-(U1-IO0-Pad36) -> Net-(U1-IO0)
Routing:
- net +3.3V: track 235.6 -> 274.5 mm, vias 2 -> 3
- net /ENC3_A: track 54.7 -> 42.4 mm, vias 2 -> 1
- net Net-(U1-IO0): track 0.00 -> 4.06 mm
Other:
- board text added: "SW1 ENCODER FACING OTHER SIDE"
- board text added: "SW2 ENCODER FACING OTHER SIDE"
- board text added: "SW3 ENCODER FACING OTHER SIDE"
- board text added: "SW4 ENCODER FACING OTHER SIDE"
