File: hardware/pcb/kicad/patternflow.kicad_pcb (KiCad board)
At the start: 2 copper layers, 74 x 132.5 mm, 35 parts, among them J1 Conn_02x08_Odd_Even, J2 Screw_Terminal_01x02, J3 Screw_Terminal_01x02, SW1 RotaryEncoder_Switch, SW2 RotaryEncoder_Switch, SW3 RotaryEncoder_Switch, SW4 RotaryEncoder_Switch, U1 ESP32-S3-DevKit-44pin

Commit message: Update PCB source to v2
Other:
- board text added: "v2.0 Open hardware · CC-BY-SA 4.0 github.com/engmung/PatternFlow"
- board text removed: "v1.0 Open hardware · CC-BY-SA 4.0 github.com/engmung/PatternFlow"
Changed lines of the file:
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@@
 		)
 	)
-	(gr_text "v1.0  \nOpen hardware · CC-BY-SA 4.0\ngithub.com/engmung/PatternFlow"
+	(gr_text "v2.0\nOpen hardware · CC-BY-SA 4.0\ngithub.com/engmung/PatternFlow"
 		(at 57.75 43.5 0)
 		(layer "F.SilkS")
@@
 	)
 	(segment
+		(start 102.5 133.07)
+		(end 99.93 130.5)
+		(width 0.2)
+		(layer "F.Cu")
+		(net "Net-(U1-IO0)")
+	)
+	(segment
+		(start 99.93 130.5)
+		(end 99.5 130.5)
+		(width 0.2)
+		(layer "F.Cu")
+		(net "Net-(U1-IO0)")
+	)
+	(segment
 		(start 94.75 128.25)
 		(end 94.75 114)
@@
 		(net "/HUB_E")
 	)
-	(segment
-		(start 102.5 133.07)
-		(end 99.93 130.5)
-		(width 0.2)
-		(layer "F.Cu")
-		(net "Net-(U1-IO0)")
-	)
-	(segment
-		(start 99.93 130.5)
-		(end 99.5 130.5)
-		(width 0.2)
-		(layer "F.Cu")
-		(net "Net-(U1-IO0)")
-	)
 	(zone

Commit message: hardware: update PCB gerbers to v2
Parts:
- added C11: 1000uF/1.6V, Capacitor_THT:CP_Radial_D10.0mm_P5.00mm, F.Cu at (67.0, 146.0)
