File: hardware/pcb/kicad/patternflow.kicad_pcb (KiCad board)
At the start: 2 copper layers, 62 x 116.2 mm, 12 parts, among them J1 Conn_02x08_Odd_Even, J3 Screw_Terminal_01x02, J4 Screw_Terminal_01x02, SW1 RotaryEncoder_Switch, SW2 RotaryEncoder_Switch, SW3 RotaryEncoder_Switch, SW4 RotaryEncoder_Switch, U1 ESP32-S3-DevKit-44pin

Commit message: hardware: v3.9 - the USB-C power input comes off the board, and the 330 case gets a wired route to the DevKit
v3.0 shipped a USB1 receptacle and its R1/R2 CC pull-downs that the build
guide, the BOM and the release notes all told you to leave unpopulated, after
the delayed burnout in #221. A footprint nobody is allowed to populate is an
instruction waiting to be ignored, so all three come off the board: J4, the
screw terminal, is the only power input there is.

Nothing else moved. The Edge_Cuts and NPTH gerbers are byte-identical to v3.0,
so the outline and every mounting hole are unchanged and the v3 cases fit both
boards. ERC went from 50 violations to 34 - the twelve pin_to_pin errors were
the USB-C net, and what remains are the same off-grid endpoints the fabricated
v3.0 carried. DRC reports no errors and no schematic-parity issues.

The 330 mm case gains a pass-through between the power-bank bay and the ESP32,
so a USB-C lead reaches the DevKit's own port with the case shut - for wired
features like MIDI and OSC, not for power - plus a cable exit slot below the
battery compartment. The 256 mm variant does not carry these yet.

Regenerated for v3.9: gerbers (14 files), BOM, board renders, schematic PDF and
SVG. The gerber command in the PCB README now pins the layer list, which is
what keeps the zip to the 14 fab files rather than all 29 layers.

Co-Authored-By: Claude Opus 5 <noreply@anthropic.com>
Parts:
- removed R1, R2: 5.1k, Resistor_THT:R_Axial_DIN0207_L6.3mm_D2.5mm_P7.62mm_Horizontal
- removed USB1: TYPE-C 14P CC-2.6, patternflow:TYPE-C-TH_TYPE-C-14P-CC-2.6
- moved J4 32.1 mm to (66.6, 150.1)
- moved C11 1.82 mm to (71.7, 138.7)
Routing:
- net Net-(USB1-CC2): track 20.3 -> 0.00 mm
- net GND: track 19.4 -> 0.00 mm, vias 99 -> 97
- net Net-(USB1-CC1): track 19.0 -> 0.00 mm
- net +5V: track 5.80 -> 0.00 mm
Other:
- board text added: "hole!"
- board text added: "v3.9 Open hardware · CC-BY-SA 4.0 · github.com/engmung/Patternflow"
- board text removed: "v3.0 Open hardware · CC-BY-SA 4.0 · github.com/engmung/Patternflow"
